Commit message: fix_naming

File: P4-Map-My-World/slam_robot/urdf/my_robot.xacro (robot description, xacro)
@@ -188,5 +188,5 @@
       <origin xyz="0 0 0" rpy=" 0 0 0"/>
       <geometry>
-        <mesh filename="package://my_robot/meshes/hokuyo.dae"/>
+        <mesh filename="package://slam_robot/meshes/hokuyo.dae"/>
       </geometry>
     </visual>
